File: ampli1W.sch (KiCad schematic (older format))
At the start: 17 parts, among them P1 SMA, P2 SMA, P3 CONN_01X01, T1 ADT1.5-1, T2 T4-1-X65, U1 OPA2677

Commit message: opened and saved with Kicad 8.0.4
Parts:
- C1, C2, C3, C4, C5: symbol CP -> ampli1W-rescue:CP
- P1, P2: symbol BNC -> ampli1W-rescue:BNC
- P3: symbol CONN_01X01 -> ampli1W-rescue:CONN_01X01
- R1, R2, R3, R4, R5, R6: symbol R -> ampli1W-rescue:R
- T1, T2: symbol TRANSFO4-RESCUE-ampli1W -> ampli1W-rescue:TRANSFO4-RESCUE-ampli1W
- U1: symbol OP275-RESCUE-ampli1W -> ampli1W-rescue:OP275-RESCUE-ampli1W
Other:
- moved on the sheet: C1, C2, C3, C4, C5, P1, P2, P3, R1, R2, R3, R4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
